Commit message: urdf: update iiwa7 urdf and add a base with 0 height

File: exotica_examples/resources/robots/iiwa7.urdf (robot description, URDF)
Before this commit: robot iiwa7, 10 links, 9 joints
Links:
- removed link world
- added link base; collision box size=1 1 0; visual box size=1 1 0
Joints:
- removed joint world_iiwa_joint
- added joint base_iiwa_joint: type fixed, parent base, child iiwa_link_0, origin xyz=0.0 0.0 0.0 rpy=0.0 0.0 0.0
